File: FlightComputer/Microcontroller.kicad_sch (KiCad schematic)
At the start: 0 parts

Commit message: Various updates
Parts:
- added C15, C16, C17, C18, C21, C22: 100n, Capacitor_SMD:C_0603_1608Metric_Pad1.08x0.95mm_HandSolder, symbol Device:C_Small
- added C19: 10u, Capacitor_SMD:C_0603_1608Metric_Pad1.08x0.95mm_HandSolder, symbol Device:C_Small
- added C20: 1u, Capacitor_SMD:C_0603_1608Metric_Pad1.08x0.95mm_HandSolder, symbol Device:C_Small
- added FB1: FerriteBead_Small, symbol Device:FerriteBead_Small
- added JP1, JP2: Jumper_3_Open, symbol Jumper:Jumper_3_Open
- added R12, R13, R14, R15, R16: 10k, Resistor_SMD:R_0603_1608Metric_Pad0.98x0.95mm_HandSolder, symbol Device:R_Small
- added SW1: SW_Push, symbol Switch:SW_Push
- added U5: STM32F103RGTx, Package_QFP:LQFP-64_10x10mm_P0.5mm, symbol MCU_ST_STM32F1:STM32F103RGTx
Connections:
- new net: JP1.2 (C), R12.1
- new net: R16.1, SW1.2, U5.7 (NRST)
- new net: JP2.2 (C), R13.1
- new net +3V3: C15.1, C16.1, C17.1, C18.1, C19.1, C22.1, FB1.1, JP1.3 (B), JP2.3 (B), R14.2, R15.2, R16.2, U5.1 (VBAT), U5.19 (VDD), U5.32 (VDD), U5.48 (VDD), U5.64 (VDD)
- new net GND: C15.2, C16.2, C17.2, C18.2, C19.2, C20.2, C21.2, C22.2, JP1.1 (A), JP2.1 (A), SW1.1, U5.12 (VSSA), U5.18 (VSS), U5.31 (VSS), U5.47 (VSS), U5.63 (VSS)
- new net JTAG_NRST: U5.56 (PB4)
- new net JTAG_TCK: U5.49 (PA14)
- new net JTAG_TDI: U5.50 (PA15)
- new net JTAG_TDO: U5.55 (PB3)
- new net JTAG_TMS: U5.46 (PA13)
- new net SCL: R14.1, U5.29 (PB10)
- new net SDA: R15.1, U5.30 (PB11)
- new net VDDA: C20.1, C21.1, FB1.2, U5.13 (VDDA)
- new net dIO_INT1_ACCEL: U5.4 (PC15)
- new net dIO_INT1_GYRO: U5.3 (PC14)
- new net dIO_INT2_ACCEL: U5.5 (PD0)
- new net dIO_INT2_GYRO: U5.2 (PC13)
- new net dIO_USB_DN: U5.45 (PA12)
- new net dIO_USB_DP: U5.44 (PA11)
- new net dI_BOOT0: R12.2, U5.60 (BOOT0)
- new net dI_BOOT1: R13.2, U5.28 (PB2)
Other:
- note added: "Boot Mode Select"
- note added: "Decoupling Caps"
- note added: "VDD"
- note added: "VDDA"
- company: (none) -> MD
- title: (none) -> Flight Computer: Microcontroller
