File: FlightComputer/Sensors.kicad_sch (KiCad schematic)
At the start: 12 parts

Commit message: Various updates
Parts:
- U3: footprint (none) -> CustomKicadFootprints:BMI088
Other:
- company: (none) -> MD
- title: (none) -> Flight Computer: Sensors
Changed lines of the file:
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@@
 	(generator_version "9.0")
 	(paper "A4")
+	(title_block
+		(title "Flight Computer: Sensors")
+		(date "2026-01-19")
+		(rev "A0.1")
+		(company "MD")
+	)
 	(rectangle
 		(start 12.7 12.7)
@@
 			)
 		)
-		(property "Footprint" ""
+		(property "Footprint" "CustomKicadFootprints:BMI088"
 			(at 180.34 49.53 0)
 			(effects
